File: hardware/quadcopter.sch (EAGLE design)
At the start: 63 parts, among them J1 AVR_SPI_PRG_6NS, J3 HEADER-10POSTH-254X10, J4 HEADER-4POS-0.1IN-FEMALE-SMD-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, J6 HEADER-4POS-0.1IN-FEMALE, Q3 MOSFET-FET-SI2302CDS-T1-E3CT-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, Q4 MOSFET-FET-SI2302CDS-T1-E3CT-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, Q5 MOSFET-FET-SI2302CDS-T1-E3CT-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, Q6 MOSFET-FET-SI2302CDS-T1-E3CT-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, U1 ATMEGA128RFA1, U2 IMU-LSM6DSOXTR-497-18367-1-ND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

Commit message: fixing many issues from quick check
Parts:
- renumbered MOTOR_PAD_1 to MP1, MOTOR_PAD_2 to MP2, MOTOR_PAD_3 to MP3, MOTOR_PAD_4 to MP4
Changed lines of the file:
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@@
 <part name="R5" library="quadparts_prebuilt_2022" deviceset="RESISTOR_" device="SMD-2012-0805-10K" value="10K"/>
 <part name="P+11" library="quadparts_prebuilt_2022" deviceset="VBAT" device=""/>
-<part name="MOTOR_PAD_1" library="quadparts_prebuilt_2022" deviceset="MOTOR_PADS_GND" device="-MOLEX-SMD"/>
+<part name="MP1" library="quadparts_prebuilt_2022" deviceset="MOTOR_PADS_GND" device="-MOLEX-SMD"/>
 <part name="GND24" library="quadparts_prebuilt_2022" deviceset="BAT_GND" device=""/>
 <part name="D5" library="quadparts_prebuilt_2022" deviceset="DIODE-SCHOTTKY_" device="-SMD-SOD123" package3d_urn="urn:adsk.eagle:package:11793366/1" value="360mV"/>
@@
 <part name="GND26" library="quadparts_prebuilt_2022" deviceset="BAT_GND" device=""/>
 <part name="P+12" library="quadparts_prebuilt_2022" deviceset="VBAT" device=""/>
-<part name="MOTOR_PAD_2" library="quadparts_prebuilt_2022" deviceset="MOTOR_PADS_GND" device="-MOLEX-SMD"/>
+<part name="MP2" library="quadparts_prebuilt_2022" deviceset="MOTOR_PADS_GND" device="-MOLEX-SMD"/>
 <part name="GND27" library="quadparts_prebuilt_2022" deviceset="BAT_GND" device=""/>
 <part name="D6" library="quadparts_prebuilt_2022" deviceset="DIODE-SCHOTTKY_" device="-SMD-SOD123" package3d_urn="urn:adsk.eagle:package:11793366/1" value="360mV"/>
@@
 <part name="GND29" library="quadparts_prebuilt_2022" deviceset="BAT_GND" device=""/>
 <part name="P+13" library="quadparts_prebuilt_2022" deviceset="VBAT" device=""/>
-<part name="MOTOR_PAD_3" library="quadparts_prebuilt_2022" deviceset="MOTOR_PADS_GND" device="-MOLEX-SMD"/>
+<part name="MP3" library="quadparts_prebuilt_2022" deviceset="MOTOR_PADS_GND" device="-MOLEX-SMD"/>
 <part name="GND30" library="quadparts_prebuilt_2022" deviceset="BAT_GND" device=""/>
 <part name="D7" library="quadparts_prebuilt_2022" deviceset="DIODE-SCHOTTKY_" device="-SMD-SOD123" package3d_urn="urn:adsk.eagle:package:11793366/1" value="360mV"/>
@@
 <part name="GND32" library="quadparts_prebuilt_2022" deviceset="BAT_GND" device=""/>
 <part name="P+14" library="quadparts_prebuilt_2022" deviceset="VBAT" device=""/>
-<part name="MOTOR_PAD_4" library="quadparts_prebuilt_2022" deviceset="MOTOR_PADS_GND" device="-MOLEX-SMD"/>
+<part name="MP4" library="quadparts_prebuilt_2022" deviceset="MOTOR_PADS_GND" device="-MOLEX-SMD"/>
 <part name="GND33" library="quadparts_prebuilt_2022" deviceset="BAT_GND" device=""/>
 <part name="D8" library="quadparts_prebuilt_2022" deviceset="DIODE-SCHOTTKY_" device="-SMD-SOD123" package3d_urn="urn:adsk.eagle:package:11793366/1" value="360mV"/>
@@
 <attribute name="VALUE" x="-198.12" y="-40.64" size="1.778" layer="96" rot="R180" align="center"/>
 </instance>
-<instance part="MOTOR_PAD_1" gate="G$1" x="-190.5" y="-63.5" smashed="yes">
+<instance part="MP1" gate="G$1" x="-190.5" y="-63.5" smashed="yes">
 <attribute name="NAME" x="-193.04" y="-55.88" size="0.8128" layer="95"/>
 </instance>
@@
 <attribute name="VALUE" x="-154.94" y="-40.64" size="1.778" layer="96" rot="R180" align="center"/>
 </instance>
-<instance part="MOTOR_PAD_2" gate="G$1" x="-147.32" y="-63.5" smashed="yes">
+<instance part="MP2" gate="G$1" x="-147.32" y="-63.5" smashed="yes">
 <attribute name="NAME" x="-149.86" y="-55.88" size="0.8128" layer="95"/>
 </instance>
@@
 <attribute name="VALUE" x="-114.3" y="-40.64" size="1.778" layer="96" rot="R180" align="center"/>
 </instance>
-<instance part="MOTOR_PAD_3" gate="G$1" x="-106.68" y="-63.5" smashed="yes">
+<instance part="MP3" gate="G$1" x="-106.68" y="-63.5" smashed="yes">
 <attribute name="NAME" x="-109.22" y="-55.88" size="0.8128" layer="95"/>
 </instance>
@@
 <attribute name="VALUE" x="-68.58" y="-40.64" size="1.778" layer="96" rot="R180" align="center"/>
 </instance>
-<instance part="MOTOR_PAD_4" gate="G$1" x="-60.96" y="-63.5" smashed="yes">
+<instance part="MP4" gate="G$1" x="-60.96" y="-63.5" smashed="yes">
 <attribute name="NAME" x="-63.5" y="-55.88" size="0.8128" layer="95"/>
 </instance>
@@
 <wire x1="-180.34" y1="-50.8" x2="-180.34" y2="-58.42" width="0.1524" layer="91"/>
 <wire x1="-180.34" y1="-58.42" x2="-182.88" y2="-58.42" width="0.1524" layer="91"/>
-<pinref part="MOTOR_PAD_1" gate="G$1" pin="V+"/>
+<pinref part="MP1" gate="G$1" pin="V+"/>
 <wire x1="-180.34" y1="-50.8" x2="-170.18" y2="-50.8" width="0.1524" layer="91"/>
 <junction x="-180.34" y="-50.8"/>
@@
 <wire x1="-137.16" y1="-50.8" x2="-137.16" y2="-58.42" width="0.1524" layer="91"/>
 <wire x1="-137.16" y1="-58.42" x2="-139.7" y2="-58.42" width="0.1524" layer="91"/>
-<pinref part="MOTOR_PAD_2" gate="G$1" pin="V+"/>
+<pinref part="MP2" gate="G$1" pin="V+"/>
 <wire x1="-137.16" y1="-50.8" x2="-127" y2="-50.8" width="0.1524" layer="91"/>
 <junction x="-137.16" y="-50.8"/>
@@
 <wire x1="-96.52" y1="-50.8" x2="-96.52" y2="-58.42" width="0.1524" layer="91"/>
 <wire x1="-96.52" y1="-58.42" x2="-99.06" y2="-58.42" width="0.1524" layer="91"/>
-<pinref part="MOTOR_PAD_3" gate="G$1" pin="V+"/>
+<pinref part="MP3" gate="G$1" pin="V+"/>
 <wire x1="-96.52" y1="-50.8" x2="-86.36" y2="-50.8" width="0.1524" layer="91"/>
 <junction x="-96.52" y="-50.8"/>
@@
 <wire x1="-50.8" y1="-50.8" x2="-50.8" y2="-58.42" width="0.1524" layer="91"/>
 <wire x1="-50.8" y1="-58.42" x2="-53.34" y2="-58.42" width="0.1524" layer="91"/>
-<pinref part="MOTOR_PAD_4" gate="G$1" pin="V+"/>
+<pinref part="MP4" gate="G$1" pin="V+"/>
 <wire x1="-50.8" y1="-50.8" x2="-40.64" y2="-50.8" width="0.1524" layer="91"/>
 <junction x="-50.8" y="-50.8"/>
@@
 <net name="BAT_GND" class="0">
 <segment>
-<pinref part="MOTOR_PAD_1" gate="G$1" pin="GND"/>
+<pinref part="MP1" gate="G$1" pin="GND"/>
 <pinref part="GND24" gate="1" pin="BAT_GND"/>
 </segment>
 <segment>
-<pinref part="MOTOR_PAD_2" gate="G$1" pin="GND"/>
+<pinref part="MP2" gate="G$1" pin="GND"/>
 <pinref part="GND27" gate="1" pin="BAT_GND"/>
 </segment>
@@
 </segment>
 <segment>
-<pinref part="MOTOR_PAD_3" gate="G$1" pin="GND"/>
+<pinref part="MP3" gate="G$1" pin="GND"/>
 <pinref part="GND30" gate="1" pin="BAT_GND"/>
 </segment>
@@
 </segment>
 <segment>
-<pinref part="MOTOR_PAD_4" gate="G$1" pin="GND"/>
+<pinref part="MP4" gate="G$1" pin="GND"/>
 <pinref part="GND33" gate="1" pin="BAT_GND"/>
 </segment>
@@
 <wire x1="-170.18" y1="-58.42" x2="-170.18" y2="-63.5" width="0.1524" layer="91"/>
 <pinref part="Q3" gate="G$1" pin="D"/>
-<pinref part="MOTOR_PAD_1" gate="G$1" pin="V-"/>
+<pinref part="MP1" gate="G$1" pin="V-"/>
 <wire x1="-170.18" y1="-63.5" x2="-170.18" y2="-76.2" width="0.1524" layer="91"/>
 <wire x1="-182.88" y1="-63.5" x2="-170.18" y2="-63.5" width="0.1524" layer="91"/>
@@
 <wire x1="-127" y1="-58.42" x2="-127" y2="-63.5" width="0.1524" layer="91"/>
 <pinref part="Q4" gate="G$1" pin="D"/>
-<pinref part="MOTOR_PAD_2" gate="G$1" pin="V-"/>
+<pinref part="MP2" gate="G$1" pin="V-"/>
 <wire x1="-127" y1="-63.5" x2="-127" y2="-76.2" width="0.1524" layer="91"/>
 <wire x1="-139.7" y1="-63.5" x2="-127" y2="-63.5" width="0.1524" layer="91"/>
@@
 <wire x1="-86.36" y1="-58.42" x2="-86.36" y2="-63.5" width="0.1524" layer="91"/>
 <pinref part="Q5" gate="G$1" pin="D"/>
-<pinref part="MOTOR_PAD_3" gate="G$1" pin="V-"/>
+<pinref part="MP3" gate="G$1" pin="V-"/>
 <wire x1="-86.36" y1="-63.5" x2="-86.36" y2="-76.2" width="0.1524" layer="91"/>
 <wire x1="-99.06" y1="-63.5" x2="-86.36" y2="-63.5" width="0.1524" layer="91"/>
@@
 <wire x1="-40.64" y1="-58.42" x2="-40.64" y2="-63.5" width="0.1524" layer="91"/>
 <pinref part="Q6" gate="G$1" pin="D"/>
-<pinref part="MOTOR_PAD_4" gate="G$1" pin="V-"/>
+<pinref part="MP4" gate="G$1" pin="V-"/>
 <wire x1="-40.64" y1="-63.5" x2="-40.64" y2="-76.2" width="0.1524" layer="91"/>
 <wire x1="-53.34" y1="-63.5" x2="-40.64" y2="-63.5" width="0.1524" layer="91"/>

Commit message: fixed a bunch of routing issues/vias, added logo
Parts:
- removed J1: AVR_SPI_PRG_6NS, quadparts_prebuilt_2022:AVR_SPI_PRG_6NS
- added H1, H2, H3, H4: MOUNTING_HOLE-2-56, quadparts_prebuilt_2022:MOUNTING_HOLE-2-56
- added J2: AVR_SPI_PRG_6-SMD, quadparts_prebuilt_2022:AVR_SPI_PRG_6-SMD
- added U$2: PIDLOGO, logo:PIDLOGO
Connections:
- net GND: now also J2.6; no longer J1.6
- net MISO: now also J2.1; no longer J1.1
- net MOSI: now also J2.4; no longer J1.4
- net RESET: now also J2.5; no longer J1.5
- net SCK: now also J2.3; no longer J1.3
Changed lines of the file:
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@@
 <class number="0" name="default" width="0" drill="0">
 </class>
-<class number="1" name="HIGH-I" width="0" drill="0">
+<class number="1" name="HIGH-I" width="0.381" drill="0">
 </class>
-<class number="2" name="RF" width="0" drill="0">
+<class number="3" name="POWER" width="0" drill="0">
+</class>
+<class number="4" name="RFSIG" width="0" drill="0">
 </class>
 </classes>
@@
 <part name="GND13" library="quadparts_prebuilt_2022" deviceset="GND" device=""/>
 <part name="GND14" library="quadparts_prebuilt_2022" deviceset="GND" device=""/>
-<part name="J1" library="quadparts_prebuilt_2022" deviceset="AVR_SPI_PRG_6" device="NS"/>
-<part name="GND15" library="quadparts_prebuilt_2022" deviceset="GND" device=""/>
 <part name="U2" library="custom_v9" library_urn="urn:adsk.wipprod:fs.file:vf.hOpq96TzSi2cy5Li20AtXQ" deviceset="IMU-LSM6DSOXTR-497-18367-1-ND" device="497-18367-1-ND"/>
 <part name="GND16" library="quadparts_prebuilt_2022" deviceset="GND" device=""/>
@@
 <part name="GND40" library="quadparts_prebuilt_2022" deviceset="GND" device=""/>
 <part name="GND41" library="quadparts_prebuilt_2022" deviceset="GND" device=""/>
+<part name="J2" library="quadparts_prebuilt_2022" deviceset="AVR_SPI_PRG_6" device="-SMD"/>
+<part name="GND44" library="quadparts_prebuilt_2022" deviceset="GND" device=""/>
+<part name="H1" library="quadparts_prebuilt_2022" deviceset="MOUNTING_HOLE" device="-2-56"/>
+<part name="H2" library="quadparts_prebuilt_2022" deviceset="MOUNTING_HOLE" device="-2-56"/>
+<part name="H3" library="quadparts_prebuilt_2022" deviceset="MOUNTING_HOLE" device="-2-56"/>
+<part name="H4" library="quadparts_prebuilt_2022" deviceset="MOUNTING_HOLE" device="-2-56"/>
+<part name="U$2" library="logo" deviceset="PIDLOGO" device=""/>
 </parts>
 <sheets>
@@
 <attribute name="VALUE" x="-111.76" y="-7.62" size="1.778" layer="96" align="center"/>
 </instance>
-<instance part="J1" gate="G$1" x="20.32" y="83.82" smashed="yes">
-<attribute name="VALUE" x="16.256" y="76.2" size="1.778" layer="96"/>
-<attribute name="NAME" x="16.002" y="89.662" size="1.778" layer="95"/>
-</instance>
-<instance part="GND15" gate="1" x="30.48" y="76.2" smashed="yes">
-<attribute name="VALUE" x="30.48" y="73.66" size="1.778" layer="96" align="center"/>
-</instance>
 <instance part="U2" gate="G$1" x="142.24" y="119.38" smashed="yes">
 <attribute name="NAME" x="137.16" y="132.08" size="1.778" layer="95"/>
@@
 <instance part="GND41" gate="1" x="127" y="-38.1" smashed="yes">
 <attribute name="VALUE" x="127" y="-40.64" size="1.778" layer="96" align="center"/>
+</instance>
+<instance part="J2" gate="G$1" x="20.32" y="101.6" smashed="yes">
+<attribute name="VALUE" x="16.256" y="93.98" size="1.778" layer="96"/>
+<attribute name="NAME" x="16.002" y="107.442" size="1.778" layer="95"/>
+</instance>
+<instance part="GND44" gate="1" x="35.56" y="96.52" smashed="yes">
+<attribute name="VALUE" x="35.56" y="93.98" size="1.778" layer="96" align="center"/>
+</instance>
+<instance part="H1" gate="G$1" x="167.64" y="-78.74" smashed="yes">
+<attribute name="NAME" x="167.64" y="-77.47" size="0.9" layer="95" font="vector" align="center"/>
+<attribute name="VALUE" x="167.64" y="-80.01" size="0.9" layer="96" font="vector" align="center"/>
+</instance>
+<instance part="H2" gate="G$1" x="187.96" y="-78.74" smashed="yes">
+<attribute name="NAME" x="187.96" y="-77.47" size="0.9" layer="95" font="vector" align="center"/>
+<attribute name="VALUE" x="187.96" y="-80.01" size="0.9" layer="96" font="vector" align="center"/>
+</instance>
+<instance part="H3" gate="G$1" x="205.74" y="-78.74" smashed="yes">
+<attribute name="NAME" x="205.74" y="-77.47" size="0.9" layer="95" font="vector" align="center"/>
+<attribute name="VALUE" x="205.74" y="-80.01" size="0.9" layer="96" font="vector" align="center"/>
+</instance>
+<instance part="H4" gate="G$1" x="154.94" y="-78.74" smashed="yes">
+<attribute name="NAME" x="154.94" y="-77.47" size="0.9" layer="95" font="vector" align="center"/>
+<attribute name="VALUE" x="154.94" y="-80.01" size="0.9" layer="96" font="vector" align="center"/>
+</instance>
+<instance part="U$2" gate="G$1" x="88.9" y="-109.22" smashed="yes">
+<attribute name="NAME" x="86.36" y="-106.68" size="1.778" layer="94" font="vector"/>
 </instance>
 </instances>
@@
 </segment>
 </net>
-<net name="GND" class="0">
+<net name="GND" class="3">
 <segment>
 <pinref part="GND1" gate="1" pin="GND"/>
@@
 </segment>
 <segment>
-<pinref part="J1" gate="G$1" pin="6"/>
-<wire x1="30.48" y1="81.28" x2="30.48" y2="78.74" width="0.1524" layer="91"/>
-<pinref part="GND15" gate="1" pin="GND"/>
-</segment>
-<segment>
 <wire x1="124.46" y1="116.84" x2="119.38" y2="116.84" width="0.1524" layer="91"/>
 <pinref part="GND16" gate="1" pin="GND"/>
@@
 <pinref part="R12" gate="G$1" pin="1"/>
 </segment>
+<segment>
+<pinref part="J2" gate="G$1" pin="6"/>
+<wire x1="30.48" y1="99.06" x2="35.56" y2="99.06" width="0.1524" layer="91"/>
+<pinref part="GND44" gate="1" pin="GND"/>
+</segment>
 </net>
 <net name="PG0" class="0">
@@
 </segment>
 </net>
-<net name="3V" class="0">
+<net name="3V" class="3">
 <segment>
 <pinref part="P+1" gate="G$1" pin="3V"/>
@@
 </segment>
 <segment>
-<pinref part="J1" gate="G$1" pin="3"/>
-<wire x1="12.7" y1="83.82" x2="7.62" y2="83.82" width="0.1524" layer="91"/>
-<label x="7.62" y="83.82" size="1.778" layer="95" rot="R180" xref="yes"/>
+<pinref part="J2" gate="G$1" pin="3"/>
+<wire x1="12.7" y1="101.6" x2="7.62" y2="101.6" width="0.1524" layer="91"/>
+<label x="7.62" y="101.6" size="1.778" layer="95" rot="MR0" xref="yes"/>
 </segment>
 </net>
@@
 </segment>
 <segment>
-<pinref part="J1" gate="G$1" pin="4"/>
-<wire x1="30.48" y1="83.82" x2="35.56" y2="83.82" width="0.1524" layer="91"/>
-<label x="35.56" y="83.82" size="1.778" layer="95" xref="yes"/>
+<pinref part="J2" gate="G$1" pin="4"/>
+<wire x1="30.48" y1="101.6" x2="35.56" y2="101.6" width="0.1524" layer="91"/>
+<label x="35.56" y="101.6" size="1.778" layer="95" xref="yes"/>
 </segment>
 </net>
@@
 </segment>
 <segment>
-<pinref part="J1" gate="G$1" pin="1"/>
-<wire x1="12.7" y1="86.36" x2="7.62" y2="86.36" width="0.1524" layer="91"/>
-<label x="7.62" y="86.36" size="1.778" layer="95" rot="R180" xref="yes"/>
+<pinref part="J2" gate="G$1" pin="1"/>
+<wire x1="12.7" y1="104.14" x2="7.62" y2="104.14" width="0.1524" layer="91"/>
+<label x="7.62" y="104.14" size="1.778" layer="95" rot="MR0" xref="yes"/>
 </segment>
 </net>
@@
 </segment>
 <segment>
-<pinref part="J1" gate="G$1" pin="5"/>
-<wire x1="12.7" y1="81.28" x2="7.62" y2="81.28" width="0.1524" layer="91"/>
-<label x="7.62" y="81.28" size="1.778" layer="95" rot="R180" xref="yes"/>
-</segment>
-<segment>
 <wire x1="25.4" y1="38.1" x2="30.48" y2="38.1" width="0.1524" layer="91"/>
 <label x="30.48" y="38.1" size="1.778" layer="95" xref="yes"/>
 <pinref part="C12" gate="G$1" pin="1"/>
+</segment>
+<segment>
+<pinref part="J2" gate="G$1" pin="5"/>
+<wire x1="12.7" y1="99.06" x2="7.62" y2="99.06" width="0.1524" layer="91"/>
+<label x="7.62" y="99.06" size="1.778" layer="95" rot="MR0" xref="yes"/>
 </segment>
 </net>
@@
 <wire x1="-81.28" y1="66.04" x2="-60.96" y2="66.04" width="0.1524" layer="91"/>
 <pinref part="B1" gate="G$1" pin="OUT1"/>
-<label x="-104.14" y="60.96" size="1.778" layer="95"/>
+<label x="-109.22" y="63.5" size="1.778" layer="95"/>
 </segment>
 </net>
@@
 <wire x1="-101.6" y1="60.96" x2="-111.76" y2="60.96" width="0.1524" layer="91"/>
 <pinref part="U1" gate="G$1" pin="RFN"/>
-<label x="-99.06" y="55.88" size="1.778" layer="95"/>
-</segment>
-</net>
-<net name="N$7" class="2">
+<label x="-101.6" y="58.42" size="1.778" layer="95"/>
+</segment>
+</net>
+<net name="N$7" class="4">
 <segment>
 <pinref part="B1" gate="G$1" pin="IN"/>
@@
 </segment>
 </net>
-<net name="BAT_GND" class="0">
+<net name="BAT_GND" class="1">
 <segment>
 <pinref part="MP1" gate="G$1" pin="GND"/>
@@
 </segment>
 </net>
-<net name="N$18" class="1">
+<net name="N$18" class="0">
 <segment>
 <wire x1="-170.18" y1="-58.42" x2="-170.18" y2="-63.5" width="0.1524" layer="91"/>
@@
 </segment>
 </net>
-<net name="N$19" class="1">
+<net name="N$19" class="0">
 <segment>
 <wire x1="-127" y1="-58.42" x2="-127" y2="-63.5" width="0.1524" layer="91"/>
@@
 </segment>
 </net>
-<net name="N$20" class="1">
+<net name="N$20" class="0">
 <segment>
 <wire x1="-86.36" y1="-58.42" x2="-86.36" y2="-63.5" width="0.1524" layer="91"/>
@@
 </segment>
 </net>
-<net name="N$21" class="1">
+<net name="N$21" class="0">
 <segment>
 <wire x1="-40.64" y1="-58.42" x2="-40.64" y2="-63.5" width="0.1524" layer="91"/>

Commit message: fixed a bunch of routing issues/vias, added logo
Parts:
- renumbered U$2 to LOGO
Changed lines of the file:
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@@
 <part name="H3" library="quadparts_prebuilt_2022" deviceset="MOUNTING_HOLE" device="-2-56"/>
 <part name="H4" library="quadparts_prebuilt_2022" deviceset="MOUNTING_HOLE" device="-2-56"/>
-<part name="U$2" library="logo" deviceset="PIDLOGO" device=""/>
+<part name="LOGO" library="logo" deviceset="PIDLOGO" device=""/>
 </parts>
 <sheets>
@@
 <attribute name="VALUE" x="154.94" y="-80.01" size="0.9" layer="96" font="vector" align="center"/>
 </instance>
-<instance part="U$2" gate="G$1" x="88.9" y="-109.22" smashed="yes">
+<instance part="LOGO" gate="G$1" x="88.9" y="-109.22" smashed="yes">
 <attribute name="NAME" x="86.36" y="-106.68" size="1.778" layer="94" font="vector"/>
 </instance>
@@
 </segment>
 </net>
-<net name="N$3" class="0">
-<segment>
-</segment>
-</net>
