File: hardware/quadcopter.sch (EAGLE design)
At the start: 68 parts, among them J2 AVR_SPI_PRG_6-SMD, J3 HEADER-10POSTH-254X10, J4 HEADER-4POS-0.1IN-FEMALE-SMD-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, J6 HEADER-4POS-0.1IN-FEMALE, Q3 MOSFET-FET-SI2302CDS-T1-E3CT-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, Q4 MOSFET-FET-SI2302CDS-T1-E3CT-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, Q5 MOSFET-FET-SI2302CDS-T1-E3CT-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, Q6 MOSFET-FET-SI2302CDS-T1-E3CT-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, U1 ATMEGA128RFA1, U2 IMU-LSM6DSOXTR-497-18367-1-ND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

Commit message: final manufacturing (hopefully) :)
Parts:
- removed C11: 47uF, quadparts_prebuilt_2022:CAPACITOR-POL_47UF-SMD-1206-TAJA
Connections:
- net BAT_GND: no longer C11.-
- net N$18: no longer C11.+
Changed lines of the file:
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@@
 <part name="B2" library="quadparts_prebuilt_2022" deviceset="BATTERY" device="-SCREW-TERMINAL"/>
 <part name="C14" library="quadparts_prebuilt_2022" deviceset="CAPACITOR-POL_" device="47UF-SMD-1206-TAJA" package3d_urn="urn:adsk.eagle:package:11793387/1" value="47uF"/>
-<part name="C11" library="quadparts_prebuilt_2022" deviceset="CAPACITOR-POL_" device="47UF-SMD-1206-TAJA" package3d_urn="urn:adsk.eagle:package:11793387/1" value="47uF"/>
 <part name="GND36" library="quadparts_prebuilt_2022" deviceset="GND" device=""/>
 <part name="J6" library="quadparts_prebuilt_2022" deviceset="HEADER-4POS" device="-0.1IN-FEMALE" package3d_urn="urn:adsk.eagle:package:10071419/1"/>
@@
 <attribute name="NAME" x="-9.906" y="-47.879" size="1.778" layer="95"/>
 </instance>
-<instance part="C11" gate="G$1" x="-162.56" y="-86.36" smashed="yes">
-<attribute name="VALUE" x="-166.116" y="-88.519" size="1.778" layer="96"/>
-<attribute name="NAME" x="-162.306" y="-85.979" size="1.778" layer="95"/>
-</instance>
 <instance part="GND36" gate="1" x="167.64" y="132.08" smashed="yes">
 <attribute name="VALUE" x="167.64" y="129.54" size="1.778" layer="96" align="center"/>
@@
 <label x="76.2" y="-50.8" size="1.778" layer="95" rot="MR0" xref="yes"/>
 <pinref part="L4" gate="G$1" pin="A"/>
+</segment>
+</net>
+<net name="N$3" class="0">
+<segment>
 </segment>
 </net>
@@
 <wire x1="-170.18" y1="-86.36" x2="-170.18" y2="-101.6" width="0.1524" layer="91"/>
 <pinref part="GND26" gate="1" pin="BAT_GND"/>
-<wire x1="-162.56" y1="-91.44" x2="-162.56" y2="-101.6" width="0.1524" layer="91"/>
-<wire x1="-162.56" y1="-101.6" x2="-170.18" y2="-101.6" width="0.1524" layer="91"/>
-<junction x="-170.18" y="-101.6"/>
-<pinref part="C11" gate="G$1" pin="-"/>
 </segment>
 <segment>
@@
 <wire x1="-170.18" y1="-63.5" x2="-170.18" y2="-76.2" width="0.1524" layer="91"/>
 <wire x1="-182.88" y1="-63.5" x2="-170.18" y2="-63.5" width="0.1524" layer="91"/>
-<wire x1="-170.18" y1="-76.2" x2="-162.56" y2="-76.2" width="0.1524" layer="91"/>
-<wire x1="-162.56" y1="-76.2" x2="-162.56" y2="-83.82" width="0.1524" layer="91"/>
 <junction x="-170.18" y="-63.5"/>
-<junction x="-170.18" y="-76.2"/>
 <pinref part="D5" gate="G$1" pin="A"/>
-<pinref part="C11" gate="G$1" pin="+"/>
-</segment>
-</net>
+</segment>
+</net>
