File: hardware/quadcopter.brd (EAGLE design)
At the start: 132 x 132 mm, 69 parts, among them J2 AVR_SPI_PRG_6-SMD, J3 HEADER-10POSTH-254X10, J4 HEADER-4POS-0.1IN-FEMALE-SMD-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, J6 HEADER-4POS-0.1IN-FEMALE, Q3 MOSFET-FET-SI2302CDS-T1-E3CT-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, Q4 MOSFET-FET-SI2302CDS-T1-E3CT-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, Q5 MOSFET-FET-SI2302CDS-T1-E3CT-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, Q6 MOSFET-FET-SI2302CDS-T1-E3CT-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, U1 ATMEGA128RFA1, U2 IMU-LSM6DSOXTR-497-18367-1-ND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

Commit message: final manufacturing (hopefully) :)
Parts:
- removed C11: 47uF, quadparts_prebuilt_2022:CAPMP3216X180
- moved D7 12.8 mm to (-26.0, 27.0)
- moved Q3 7.28 mm to (29.0, -22.0), turned to 270 degrees
- moved D5 7.07 mm to (37.0, -21.0)
- moved Q5 1.00 mm to (-33.0, 24.0), turned to 0 degrees
Connections:
- net BAT_GND: no longer C11.2
- net N$18: no longer C11.1
Routing:
- net VBAT: track 22.6 -> 53.9 mm, vias 12 -> 10
- net N$18: track 21.5 -> 11.2 mm
- net PWM3: track 129.7 -> 121.1 mm, vias 3 -> 4
- net BAT_GND: track 53.4 -> 45.5 mm
- net PWM1: track 97.6 -> 91.3 mm
- net N$20: track 15.5 -> 10.8 mm
- net N$19: track 10.8 -> 12.0 mm

Commit message: :)
Parts:
- moved D5 1.00 mm to (36.0, -21.0)
Routing:
- net BAT_GND: track 45.5 -> 44.1 mm
- net N$18: track 11.2 -> 10.6 mm

Commit message: :D
Parts:
- moved C14 6.50 mm to (-21.0, -23.0), turned to 90 degrees
- moved C17 2.24 mm to (-15.0, -27.8)
Routing:
- net BAT_GND: track 44.1 -> 48.2 mm, vias 18 -> 17
- net 3V: track 92.8 -> 90.6 mm
- net GND: track 66.7 -> 67.7 mm
- net PWM4: track 112.9 -> 112.0 mm
- net PWM2: track 159.9 -> 160.8 mm

Commit message: :) :D ;)
Routing:
- net 3V: track 90.6 -> 93.2 mm, vias 13 -> 12
Changed lines of the file:
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@@
 <vertex x="-21.746" y="-17.394790625"/>
 </polygon>
-<wire x1="-19.955" y1="18" x2="-21.0994" y2="18" width="0.254" layer="1"/>
-<wire x1="-4.9984375" y1="-1.895" x2="-4.996403125" y2="-3.060084375" width="0.254" layer="1"/>
-<wire x1="-4.9984375" y1="-1.895" x2="-4.9984375" y2="-1.894996875" width="0.254" layer="1"/>
-<wire x1="7.395" y1="0" x2="7.4772" y2="0.0822" width="0.254" layer="1"/>
-<wire x1="7.4772" y1="0.0822" x2="8.5594" y2="-1" width="0.254" layer="1"/>
-<wire x1="-15.895" y1="-27.8" x2="-17.0594" y2="-27.8" width="0.254" layer="1"/>
-<wire x1="-18.955" y1="28" x2="-20.0994" y2="28" width="0.254" layer="1"/>
-<wire x1="-11.25" y1="6" x2="-12.0594" y2="6" width="0.254" layer="1"/>
-<wire x1="-16.455" y1="-0.7" x2="-17.5994" y2="-0.7" width="0.254" layer="1"/>
-<wire x1="-16.54" y1="-17.3" x2="-17.8621" y2="-17.3" width="0.254" layer="1"/>
-<wire x1="1.1625" y1="-0.75" x2="1.9044" y2="-0.75" width="0.254" layer="1"/>
-<wire x1="-0.5" y1="-0.95" x2="-0.5" y2="-1.6919" width="0.254" layer="1"/>
-<wire x1="0.5" y1="0.95" x2="0.5" y2="1.6919" width="0.254" layer="1"/>
-<wire x1="-13.3" y1="-20.45" x2="-12.2456" y2="-20.45" width="0.254" layer="1"/>
-<wire x1="-3.395" y1="7" x2="-4.5594" y2="7" width="0.254" layer="1"/>
+<wire x1="-19.955" y1="18" x2="-21.0994" y2="18" width="0.3048" layer="1"/>
+<wire x1="-15.895" y1="-27.8" x2="-17.0594" y2="-27.8" width="0.3048" layer="1"/>
+<wire x1="-16.455" y1="-0.7" x2="-17.5994" y2="-0.7" width="0.3048" layer="1"/>
+<wire x1="1.1625" y1="-0.75" x2="1.9044" y2="-0.75" width="0.3048" layer="1"/>
+<wire x1="-0.5" y1="-0.95" x2="-0.5" y2="-1.6919" width="0.3048" layer="1"/>
+<wire x1="0.5" y1="0.95" x2="0.5" y2="1.6919" width="0.3048" layer="1"/>
+<wire x1="-16.54" y1="-17.3" x2="-17.8621" y2="-17.3" width="0.3048" layer="1"/>
+<wire x1="-4.9984375" y1="-1.895" x2="-4.996403125" y2="-3.060084375" width="0.3048" layer="1"/>
+<wire x1="-4.9984375" y1="-1.895" x2="-4.9984375" y2="-1.894996875" width="0.3048" layer="1"/>
+<wire x1="-18.955" y1="28" x2="-20.0994" y2="28" width="0.3048" layer="1"/>
+<wire x1="-13.3" y1="-20.45" x2="-12.2456" y2="-20.45" width="0.3048" layer="1"/>
+<wire x1="-3.395" y1="7" x2="-4.5594" y2="7" width="0.3048" layer="1"/>
+<wire x1="-10.895" y1="6" x2="-11.25" y2="6" width="0.3048" layer="1"/>
 <via x="-21.0994" y="18" extent="1-16" drill="0.35">
 </via>
+<via x="-17.0594" y="-27.8" extent="1-16" drill="0.35">
+</via>
+<via x="-17.5994" y="-0.7" extent="1-16" drill="0.35">
+</via>
+<via x="1.9044" y="-0.75" extent="1-16" drill="0.35">
+</via>
+<via x="-0.5" y="-1.6919" extent="1-16" drill="0.35">
+</via>
+<via x="0.5" y="1.6919" extent="1-16" drill="0.35">
+</via>
+<via x="-17.8621" y="-17.3" extent="1-16" drill="0.35">
+</via>
 <via x="-4.996403125" y="-3.060084375" extent="1-16" drill="0.35">
 </via>
-<via x="8.5594" y="-1" extent="1-16" drill="0.35">
-</via>
-<via x="-17.0594" y="-27.8" extent="1-16" drill="0.35">
-</via>
 <via x="-20.0994" y="28" extent="1-16" drill="0.35">
 </via>
+<via x="-12.2456" y="-20.45" extent="1-16" drill="0.35">
+</via>
+<via x="-4.5594" y="7" extent="1-16" drill="0.35">
+</via>
 <via x="-12.0594" y="6" extent="1-16" drill="0.35">
 </via>
-<via x="-17.5994" y="-0.7" extent="1-16" drill="0.35">
-</via>
-<via x="-17.8621" y="-17.3" extent="1-16" drill="0.35">
-</via>
-<via x="1.9044" y="-0.75" extent="1-16" drill="0.35">
-</via>
-<via x="-0.5" y="-1.6919" extent="1-16" drill="0.35">
-</via>
-<via x="0.5" y="1.6919" extent="1-16" drill="0.35">
-</via>
-<via x="-12.2456" y="-20.45" extent="1-16" drill="0.35">
-</via>
-<via x="-4.5594" y="7" extent="1-16" drill="0.35">
-</via>
-<wire x1="-4.25" y1="13.75" x2="-3.119" y2="13.75" width="0.254" layer="1"/>
-<wire x1="-4.75" y1="14.25" x2="-4.25" y2="13.75" width="0.254" layer="1"/>
-<wire x1="-4.75" y1="16.25" x2="-4.75" y2="14.25" width="0.254" layer="1"/>
-<wire x1="-3.119" y1="16.25" x2="-4.75" y2="16.25" width="0.254" layer="1"/>
-<wire x1="-13.5" y1="-18.5" x2="-13.5" y2="-20.25" width="0.254" layer="1"/>
-<wire x1="-15.75" y1="-18.5" x2="-13.5" y2="-18.5" width="0.254" layer="1"/>
-<wire x1="-16.75" y1="-17.5" x2="-15.75" y2="-18.5" width="0.254" layer="1"/>
-<wire x1="-13.5" y1="-20.25" x2="-13.3" y2="-20.45" width="0.254" layer="1"/>
-<wire x1="-16.75" y1="-17.5" x2="-16.54" y2="-17.3" width="0.254" layer="1"/>
-<wire x1="-21" y1="27.25" x2="-20.25" y2="28" width="0.254" layer="16"/>
-<wire x1="-21" y1="18" x2="-21" y2="27.25" width="0.254" layer="16"/>
-<wire x1="-20.25" y1="28" x2="-20.0994" y2="28" width="0.254" layer="16"/>
-<wire x1="-21" y1="18" x2="-21.0994" y2="18" width="0.254" layer="16"/>
-<wire x1="-13.25" y1="-21.25" x2="-13.25" y2="-24.593434375" width="0.254" layer="16"/>
-<wire x1="-12.25" y1="-20.25" x2="-13.25" y2="-21.25" width="0.254" layer="16"/>
-<wire x1="-13.25" y1="-24.593434375" x2="-17.0594" y2="-27.8" width="0.254" layer="16"/>
-<wire x1="-12.2456" y1="-20.45" x2="-12.25" y2="-20.25" width="0.254" layer="16"/>
+<wire x1="-11.25" y1="6" x2="-12.0594" y2="6" width="0.3048" layer="1"/>
+<wire x1="-16.5" y1="-17.25" x2="-13.3" y2="-20.45" width="0.254" layer="1"/>
+<wire x1="-16.5" y1="-17.25" x2="-16.54" y2="-17.3" width="0.254" layer="1"/>
+<wire x1="5.5" y1="-1.75" x2="7.25" y2="0" width="0.254" layer="1"/>
+<wire x1="2" y1="-1.75" x2="5.5" y2="-1.75" width="0.254" layer="1"/>
+<wire x1="2" y1="-0.75" x2="2" y2="-1.75" width="0.254" layer="1"/>
+<wire x1="7.25" y1="0" x2="7.395" y2="0" width="0.254" layer="1"/>
+<wire x1="2" y1="-0.75" x2="1.9044" y2="-0.75" width="0.254" layer="1"/>
+<wire x1="-20.25" y1="26.5" x2="-20.25" y2="28" width="0.254" layer="15"/>
+<wire x1="-21" y1="25.75" x2="-20.25" y2="26.5" width="0.254" layer="15"/>
+<wire x1="-21" y1="18" x2="-21" y2="25.75" width="0.254" layer="15"/>
+<wire x1="-20.25" y1="28" x2="-20.0994" y2="28" width="0.254" layer="15"/>
+<wire x1="-21" y1="18" x2="-21.0994" y2="18" width="0.254" layer="15"/>
+<wire x1="-12.5" y1="-23.25" x2="-17" y2="-27.75" width="0.254" layer="16"/>
+<wire x1="-12.5" y1="-20.5" x2="-12.5" y2="-23.25" width="0.254" layer="16"/>
+<wire x1="-12.25" y1="-20.5" x2="-12.5" y2="-20.5" width="0.254" layer="16"/>
+<wire x1="-17" y1="-27.75" x2="-17.0594" y2="-27.8" width="0.254" layer="16"/>
+<wire x1="-12.25" y1="-20.5" x2="-12.2456" y2="-20.45" width="0.254" layer="16"/>
 <wire x1="-11.25" y1="6" x2="-11.25" y2="10.119" width="0.254" layer="1"/>
-<wire x1="-11.25" y1="6" x2="-10.895" y2="6" width="0.254" layer="1"/>
-<wire x1="-6.25" y1="7" x2="-6.25" y2="10.119" width="0.254" layer="1"/>
-<wire x1="-4.5594" y1="7" x2="-6.25" y2="7" width="0.254" layer="1"/>
-<wire x1="-14.25" y1="15.75" x2="-12.881" y2="15.75" width="0.254" layer="1"/>
-<wire x1="-17.5" y1="19" x2="-14.25" y2="15.75" width="0.254" layer="1"/>
-<wire x1="-18.5" y1="19" x2="-17.5" y2="19" width="0.254" layer="1"/>
-<wire x1="-19.5" y1="18" x2="-18.5" y2="19" width="0.254" layer="1"/>
-<wire x1="-19.955" y1="18" x2="-19.5" y2="18" width="0.254" layer="1"/>
-<wire x1="-5.75" y1="12.25" x2="-4.25" y2="13.75" width="0.254" layer="1"/>
-<wire x1="-5.75" y1="11.25" x2="-5.75" y2="12.25" width="0.254" layer="1"/>
-<wire x1="-6" y1="11.25" x2="-5.75" y2="11.25" width="0.254" layer="1"/>
-<wire x1="-6.25" y1="11" x2="-6" y2="11.25" width="0.254" layer="1"/>
-<wire x1="-6.25" y1="10.119" x2="-6.25" y2="11" width="0.254" layer="1"/>
-<wire x1="-12" y1="-21" x2="3" y2="-36" width="0.254" layer="16"/>
-<wire x1="-12" y1="-20.5" x2="-12" y2="-21" width="0.254" layer="16"/>
-<wire x1="-12.2456" y1="-20.45" x2="-12" y2="-20.5" width="0.254" layer="16"/>
+<wire x1="-6.25" y1="8.5" x2="-6.25" y2="10.119" width="0.254" layer="1"/>
+<wire x1="-4.75" y1="7" x2="-6.25" y2="8.5" width="0.254" layer="1"/>
+<wire x1="-4.75" y1="7" x2="-4.5594" y2="7" width="0.254" layer="1"/>
+<wire x1="-10.5" y1="15.75" x2="-12.881" y2="15.75" width="0.254" layer="1"/>
+<wire x1="-10.5" y1="11.75" x2="-10.5" y2="13.75" width="0.254" layer="1"/>
+<wire x1="-10.5" y1="13.75" x2="-10.5" y2="15.75" width="0.254" layer="1"/>
+<wire x1="-11.25" y1="11" x2="-10.5" y2="11.75" width="0.254" layer="1"/>
+<wire x1="-11.25" y1="10.119" x2="-11.25" y2="11" width="0.254" layer="1"/>
+<wire x1="-10.5" y1="13.75" x2="-4.75" y2="13.75" width="0.254" layer="1"/>
+<wire x1="-4.75" y1="13.75" x2="-3.119" y2="13.75" width="0.254" layer="1"/>
+<wire x1="-4.75" y1="16.25" x2="-3.119" y2="16.25" width="0.254" layer="1"/>
+<wire x1="-4.75" y1="13.75" x2="-4.75" y2="16.25" width="0.254" layer="1"/>
+<wire x1="2.5" y1="-35.5" x2="3" y2="-36" width="0.254" layer="16"/>
+<wire x1="0" y1="-35.5" x2="2.5" y2="-35.5" width="0.254" layer="16"/>
+<wire x1="-12.25" y1="-23.25" x2="0" y2="-35.5" width="0.254" layer="16"/>
+<wire x1="-12.5" y1="-23.25" x2="-12.25" y2="-23.25" width="0.254" layer="16"/>
 </signal>
 <signal name="SCK">
@@
 <wire x1="-6.4262" y1="11.5951" x2="-6.985" y2="11.5951" width="0.127" layer="2"/>
 <wire x1="-33.9471" y1="22.84095" x2="-33.95" y2="22.85" width="0.127" layer="1"/>
-<wire x1="14.31925" y1="-35.97275" x2="13.20165" y2="-35.97275" width="0.127" layer="15"/>
-<wire x1="14.3891" y1="-36.0426" x2="14.31925" y2="-35.97275" width="0.127" layer="15"/>
-<wire x1="14.5288" y1="-35.9029" x2="14.3891" y2="-36.0426" width="0.127" layer="15"/>
+<wire x1="14.45895" y1="-35.97275" x2="13.20165" y2="-35.97275" width="0.127" layer="15"/>
+<wire x1="14.5288" y1="-35.9029" x2="14.45895" y2="-35.97275" width="0.127" layer="15"/>
 <wire x1="14.5288" y1="-35.4838" x2="14.5288" y2="-35.9029" width="0.127" layer="15"/>
 <wire x1="15.15745" y1="-34.85515" x2="14.5288" y2="-35.4838" width="0.127" layer="15"/>

Commit message: final board? :)
Parts:
- moved LOGO 52.2 mm to (16.0, 32.9)
- moved J6 23.3 mm to (3.00, -27.5)
- moved J2 23.3 mm to (18.0, -24.0)
Routing:
- net MISO: track 33.9 -> 50.9 mm
- net SCK: track 38.2 -> 51.2 mm
- net MOSI: track 33.7 -> 46.3 mm
- net RESET: track 131.6 -> 142.4 mm, vias 3 -> 4
- net 3V: track 93.2 -> 101.1 mm, vias 12 -> 13
- net RX0: track 23.0 -> 30.6 mm, vias 2 -> 0
- net SDA: track 85.1 -> 80.5 mm
- net GND: track 67.7 -> 64.2 mm, vias 28 -> 26
- net LED2: track 44.9 -> 42.7 mm, vias 0 -> 2
- net TX0: track 28.1 -> 26.5 mm
- net SCL: track 85.4 -> 84.0 mm
- net N$13: track 40.1 -> 39.1 mm
